File: electronica/hardware/Circuitos/SoloPotencia/v1/Circuito_pulsos.sch (KiCad schematic (older format))
At the start: 33 parts, among them J3 Conn_01x03, J4 ACS712, P3 SALIDA_1, P4 SALIDA_2, Q10 IRF4905, Q11 IRFZ46N, Q12 IRF4905, Q13 IRFZ46N, Q14 2N2222, Q9 2N2222

Commit message: Se agregaron mediciones a la placa de potencia. Las mediciones con un informe se encuentran en ProcesoPTH/documentacion/MedicionesFuenteDePulsos
Parts:
- removed D10, D9: 1N4148, Diodes_THT:D_A-405_P7.62mm_Horizontal, symbol FuenteDePulsos-rescue:D
- removed D3, D8: 15v, Diodes_THT:D_A-405_P7.62mm_Horizontal, symbol Device:D_Zener
- removed Q10, Q12: IRF4905, Package_TO_SOT_THT:TO-220-3_Vertical, symbol Transistor_FET:IRF4905
- added Q10, Q12: TIP127, TO_SOT_Packages_THT:TO-220-3_Vertical, symbol FuenteDePulsos-rescue:TIP127
- added R25, R37: 100, Resistors_THT:R_Axial_DIN0207_L6.3mm_D2.5mm_P7.62mm_Horizontal, symbol FuenteDePulsos-rescue:R
- R24, R38: value 1k -> 330
Connections:
- wire segments 92 -> 63
Other:
- moved on the sheet: D4, D5, R38
