File: electronica/hardware/Circuitos/SoloPotencia/Actual/FuenteDePulsos.kicad_pcb (KiCad board)
At the start: 2 copper layers, 125.1 x 76.8 mm, 73 parts, among them J1 Conn_01x03, J2 Conn_01x05, J3 Conn_01x03, J4 ACS712, J5 Agujero, J6 Agujero, J7 Agujero, J8 Agujero, P3 SALIDA_1, P4 SALIDA_2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

Commit message: Se agregaron mediciones con el nuevo driver para el transistor PMOS
Other:
- board text added: "Este circuito es de la version 1, está desactualizado"
Changed lines of the file:
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@@
-(kicad_pcb (version 20171130) (host pcbnew 5.0.2-bee76a0~70~ubuntu18.04.1)
+(kicad_pcb (version 20171130) (host pcbnew 5.1.4-e60b266~84~ubuntu18.04.1)
   (general
     (thickness 1.6)
-    (drawings 5)
+    (drawings 6)
     (tracks 417)
     (zones 0)
@@
     (zone_45_only no)
     (trace_min 0.3048)
-    (segment_width 0.2)
-    (edge_width 0.15)
     (via_size 1.3208)
     (via_drill 0.7112)
@@
     (uvia_min_size 0.508)
     (uvia_min_drill 0.127)
+    (edge_width 0.15)
+    (segment_width 0.2)
     (pcb_text_width 0.3)
     (pcb_text_size 1 1)
@@
     (pad 1 np_thru_hole circle (at 0 0) (size 3.7 3.7) (drill 3.7) (layers *.Cu *.Mask))
   )
+  (gr_text "Este circuito es de la version 1, está desactualizado" (at 145.6182 42.5704) (layer Dwgs.User)
+    (effects (font (size 5 5) (thickness 1)))
+  )
   (gr_text LCI (at 113.03 129.54) (layer B.Cu)
